Commit message: some modifications for multi arm motion planning

File: ur_moveit_config/srdf/ur_macro.srdf.xacro (robot description, xacro)
@@ -16,7 +16,7 @@
     <!--GROUP STATES - Purpose - Define a named state for a particular group, in terms of joint values. This is useful to define states like 'folded arms'-->
     <group_state name="${prefix}home" group="${name}_manipulator">
+      <joint name="${prefix}shoulder_pan_joint" value="0" />
+      <joint name="${prefix}shoulder_lift_joint" value="-1.5707" />
       <joint name="${prefix}elbow_joint" value="0" />
-      <joint name="${prefix}shoulder_lift_joint" value="-1.5707" />
-      <joint name="${prefix}shoulder_pan_joint" value="0" />
       <joint name="${prefix}wrist_1_joint" value="0" />
       <joint name="${prefix}wrist_2_joint" value="0" />
@@ -24,7 +24,7 @@
     </group_state>
     <group_state name="${prefix}up" group="${name}_manipulator">
+      <joint name="${prefix}shoulder_pan_joint" value="0" />
+      <joint name="${prefix}shoulder_lift_joint" value="-1.5707" />
       <joint name="${prefix}elbow_joint" value="0" />
-      <joint name="${prefix}shoulder_lift_joint" value="-1.5707" />
-      <joint name="${prefix}shoulder_pan_joint" value="0" />
       <joint name="${prefix}wrist_1_joint" value="-1.5707" />
       <joint name="${prefix}wrist_2_joint" value="0" />
@@ -32,10 +32,10 @@
     </group_state>
     <group_state name="${prefix}test_configuration" group="${name}_manipulator">
-      <joint name="${prefix}elbow_joint" value="1.4" />
-      <joint name="${prefix}shoulder_lift_joint" value="-1.62" />
-      <joint name="${prefix}shoulder_pan_joint" value="1.54" />
-      <joint name="${prefix}wrist_1_joint" value="-1.2" />
-      <joint name="${prefix}wrist_2_joint" value="-1.6" />
-      <joint name="${prefix}wrist_3_joint" value="-0.11" />
+      <joint name="${prefix}shoulder_pan_joint" value="-0.8" />
+      <joint name="${prefix}shoulder_lift_joint" value="-1.57" />
+      <joint name="${prefix}elbow_joint" value="-1.57" />
+      <joint name="${prefix}wrist_1_joint" value="-1.57" />
+      <joint name="${prefix}wrist_2_joint" value="1.57" />
+      <joint name="${prefix}wrist_3_joint" value="0.0" />
     </group_state>
     <!--END EFFECTOR - Purpose - Represent information about an end effector.-->

Commit message: update for real robot test

File: ur_moveit_config/srdf/ur_macro.srdf.xacro (robot description, xacro)
@@ -12,5 +12,5 @@
     <!--SUBGROUPS - Groups can also be formed by referencing to already defined group names-->
     <group name="${name}_manipulator">
-      <chain base_link="${prefix}base_link" tip_link="${prefix}tool0" />
+      <chain base_link="${prefix}base_link" tip_link="${prefix}tool_tip" />
     </group>
     <!--GROUP STATES - Purpose - Define a named state for a particular group, in terms of joint values. This is useful to define states like 'folded arms'-->
@@ -39,4 +39,20 @@
       <joint name="${prefix}wrist_3_joint" value="0.0" />
     </group_state>
+    <group_state name="test_1" group="${name}_manipulator">
+      <joint name="${prefix}shoulder_pan_joint" value="0.785" />
+      <joint name="${prefix}shoulder_lift_joint" value="-1.57" />
+      <joint name="${prefix}elbow_joint" value="-1.57" />
+      <joint name="${prefix}wrist_1_joint" value="-1.57" />
+      <joint name="${prefix}wrist_2_joint" value="1.57" />
+      <joint name="${prefix}wrist_3_joint" value="0.0" />
+    </group_state>
+        <group_state name="test_2" group="${name}_manipulator">
+      <joint name="${prefix}shoulder_pan_joint" value="3.14" />
+      <joint name="${prefix}shoulder_lift_joint" value="-1.57" />
+      <joint name="${prefix}elbow_joint" value="-1.57" />
+      <joint name="${prefix}wrist_1_joint" value="-1.57" />
+      <joint name="${prefix}wrist_2_joint" value="1.57" />
+      <joint name="${prefix}wrist_3_joint" value="0.0" />
+    </group_state>
     <!--END EFFECTOR - Purpose - Represent information about an end effector.-->
     <!--VIRTUAL JOINT - Purpose - this element defines a virtual joint between a robot link and an external frame of reference (considered fixed with respect to the robot)-->
@@ -53,4 +69,6 @@
     <disable_collisions link1="${prefix}wrist_1_link" link2="${prefix}wrist_3_link" reason="Never" />
     <disable_collisions link1="${prefix}wrist_2_link" link2="${prefix}wrist_3_link" reason="Adjacent" />
+    <disable_collisions link1="${prefix}tool_base" link2="${prefix}wrist_2_link" reason="Never" />
+    <disable_collisions link1="${prefix}tool_base" link2="${prefix}wrist_3_link" reason="Adjacent" />
   </xacro:macro>
 </robot>

File: ur_moveit_config/urdf/ur.urdf.xacro (robot description, xacro)
@@ -5,4 +5,5 @@
   <!-- import main macro -->
   <xacro:include filename="$(find ur_description)/urdf/ur_macro.xacro"/>
+  <xacro:include filename="$(find mr_description)/urdf/suction_tool.xacro"/>
   <!-- possible 'ur_type' values: ur3, ur3e, ur5, ur5e, ur10, ur10e, ur16e -->
   <!-- the default value should raise an error in case this was called without defining the type -->
@@ -88,4 +89,10 @@
     <origin xyz="$(arg pose_xyz)" rpy="$(arg pose_rpy)" />          <!-- position robot in the world -->
   </xacro:ur_robot>
+  <xacro:tool_marco prefix="$(arg prefix)"/>
+  <joint name="$(arg prefix)tool0-tool" type="fixed">
+    <origin xyz="0 0 0" rpy="0 0 0"/>
+    <parent link="$(arg prefix)tool0"/>
+    <child link="$(arg prefix)tool_base"/>
+  </joint>
   <xacro:if value="$(arg sim_gazebo)">
     <!-- Gazebo plugins -->

Commit message: back to 2.2.4

File: ur_moveit_config/srdf/ur_macro.srdf.xacro (robot description, xacro)
@@ -11,47 +11,31 @@
     <!--CHAINS - When a chain is specified, all the links along the chain (including endpoints) are included in the group. Additionally, all the joints that are parents to included links are also included. This means that joints along the chain and the parent joint of the base link are included in the group-->
     <!--SUBGROUPS - Groups can also be formed by referencing to already defined group names-->
-    <group name="${name}_manipulator">
-      <chain base_link="${prefix}base_link" tip_link="${prefix}tool_tip" />
+    <group name="${prefix}${name}_manipulator">
+      <chain base_link="${prefix}base_link" tip_link="${prefix}tool0" />
     </group>
     <!--GROUP STATES - Purpose - Define a named state for a particular group, in terms of joint values. This is useful to define states like 'folded arms'-->
-    <group_state name="${prefix}home" group="${name}_manipulator">
+    <group_state name="${prefix}home" group="${prefix}${name}_manipulator">
+      <joint name="${prefix}elbow_joint" value="0" />
+      <joint name="${prefix}shoulder_lift_joint" value="-1.5707" />
       <joint name="${prefix}shoulder_pan_joint" value="0" />
-      <joint name="${prefix}shoulder_lift_joint" value="-1.5707" />
-      <joint name="${prefix}elbow_joint" value="0" />
       <joint name="${prefix}wrist_1_joint" value="0" />
       <joint name="${prefix}wrist_2_joint" value="0" />
       <joint name="${prefix}wrist_3_joint" value="0" />
     </group_state>
-    <group_state name="${prefix}up" group="${name}_manipulator">
+    <group_state name="${prefix}up" group="${prefix}${name}_manipulator">
+      <joint name="${prefix}elbow_joint" value="0" />
+      <joint name="${prefix}shoulder_lift_joint" value="-1.5707" />
       <joint name="${prefix}shoulder_pan_joint" value="0" />
-      <joint name="${prefix}shoulder_lift_joint" value="-1.5707" />
-      <joint name="${prefix}elbow_joint" value="0" />
       <joint name="${prefix}wrist_1_joint" value="-1.5707" />
       <joint name="${prefix}wrist_2_joint" value="0" />
       <joint name="${prefix}wrist_3_joint" value="0" />
     </group_state>
-    <group_state name="${prefix}test_configuration" group="${name}_manipulator">
-      <joint name="${prefix}shoulder_pan_joint" value="-0.8" />
-      <joint name="${prefix}shoulder_lift_joint" value="-1.57" />
-      <joint name="${prefix}elbow_joint" value="-1.57" />
-      <joint name="${prefix}wrist_1_joint" value="-1.57" />
-      <joint name="${prefix}wrist_2_joint" value="1.57" />
-      <joint name="${prefix}wrist_3_joint" value="0.0" />
-    </group_state>
-    <group_state name="test_1" group="${name}_manipulator">
-      <joint name="${prefix}shoulder_pan_joint" value="0.785" />
-      <joint name="${prefix}shoulder_lift_joint" value="-1.57" />
-      <joint name="${prefix}elbow_joint" value="-1.57" />
-      <joint name="${prefix}wrist_1_joint" value="-1.57" />
-      <joint name="${prefix}wrist_2_joint" value="1.57" />
-      <joint name="${prefix}wrist_3_joint" value="0.0" />
-    </group_state>
-        <group_state name="test_2" group="${name}_manipulator">
-      <joint name="${prefix}shoulder_pan_joint" value="3.14" />
-      <joint name="${prefix}shoulder_lift_joint" value="-1.57" />
-      <joint name="${prefix}elbow_joint" value="-1.57" />
-      <joint name="${prefix}wrist_1_joint" value="-1.57" />
-      <joint name="${prefix}wrist_2_joint" value="1.57" />
-      <joint name="${prefix}wrist_3_joint" value="0.0" />
+    <group_state name="${prefix}test_configuration" group="${prefix}${name}_manipulator">
+      <joint name="${prefix}elbow_joint" value="1.4" />
+      <joint name="${prefix}shoulder_lift_joint" value="-1.62" />
+      <joint name="${prefix}shoulder_pan_joint" value="1.54" />
+      <joint name="${prefix}wrist_1_joint" value="-1.2" />
+      <joint name="${prefix}wrist_2_joint" value="-1.6" />
+      <joint name="${prefix}wrist_3_joint" value="-0.11" />
     </group_state>
     <!--END EFFECTOR - Purpose - Represent information about an end effector.-->
@@ -69,6 +53,4 @@
     <disable_collisions link1="${prefix}wrist_1_link" link2="${prefix}wrist_3_link" reason="Never" />
     <disable_collisions link1="${prefix}wrist_2_link" link2="${prefix}wrist_3_link" reason="Adjacent" />
-    <disable_collisions link1="${prefix}tool_base" link2="${prefix}wrist_2_link" reason="Never" />
-    <disable_collisions link1="${prefix}tool_base" link2="${prefix}wrist_3_link" reason="Adjacent" />
   </xacro:macro>
 </robot>
